File: rowing-pcb.kicad_sch (KiCad schematic)
At the start: 0 parts

Commit message: Started project, coming back with changes soon.
Parts:
- added D1 (x2): SS110, PCM_Diode_SMD_AKL:D_SMA, symbol PCM_Diode_Schottky_AKL:SS110
- added D2, D3: LED, LED_SMD:LED_0603_1608Metric, symbol Device:LED
- added P1: USB_C_Plug_USB2.0, symbol Connector:USB_C_Plug_USB2.0
- added R1: 1.2k, PCM_Resistor_SMD_AKL:R_0603_1608Metric, symbol PCM_Resistor_AKL:R_0603
- added R2, R3: 1k, PCM_Resistor_SMD_AKL:R_0603_1608Metric, symbol PCM_Resistor_AKL:R_0603
- added TP1: Batt+, TestPoint:TestPoint_Pad_D1.0mm, symbol PCM_4ms_Connector:TestPoint
- added TP2: Batt-, TestPoint:TestPoint_Pad_D1.0mm, symbol PCM_4ms_Connector:TestPoint
- added U1: ESP32-S3-WROOM-1, RF_Module:ESP32-S3-WROOM-1, symbol RF_Module:ESP32-S3-WROOM-1
- added U2: TP4056, TP4056 (2):SOT23-8, symbol TP4056:TP4056
- added U3: AMS1117-3.3, Package_TO_SOT_SMD:SOT-223-3_TabPin2, symbol Regulator_Linear:AMS1117-3.3
- added U4: CP2102N-Axx-xQFN28, Package_DFN_QFN:QFN-28-1EP_5x5mm_P0.5mm_EP3.35x3.35mm, symbol Interface_USB:CP2102N-Axx-xQFN28
Connections:
- new net: D1.2 (A), P1.A4 (VBUS), P1.A9 (VBUS), P1.B4 (VBUS), P1.B9 (VBUS)
- new net: R1.1, U2.2 (PROG)
- new net: D3.1 (K), R3.1
- new net: R3.2, U2.6 (~{STDBY})
- new net: R2.2, U2.7 (~{CHRG})
- new net: D2.1 (K), R2.1
- new net Batt-v-read: D1.2 (A), TP1.1, U2.5 (BAT)
- new net DTR: U4.28 (~{DTR})
- new net Data+: P1.A6 (D+), U1.14 (USB_D+), U4.4 (D+)
- new net Data-: P1.A7 (D-), U1.13 (USB_D-), U4.5 (D-)
- new net GND: P1.A1 (GND), P1.A12 (GND), P1.B1 (GND), P1.B12 (GND), R1.2, TP2.1, U1.1 (GND), U1.40 (GND), U1.41 (GND), U2.1 (TEMP), U2.3 (GND), U3.1 (GND), U4.29 (GND), U4.3 (GND)
- new net P,+3.3: U1.2 (3V3), U3.2 (VO)
- new net RTS: U4.24 (~{RTS})
- new net RXD: U4.26 (TXD)
- new net TXD: U4.25 (RXD)
- new net VCC: D1.1 (K), D1.1 (K), D2.2 (A), D3.2 (A), U2.4 (VCC), U3.3 (VI), U4.7 (VREGIN), U4.8 (VBUS)
- no-connect marks 0 -> 22
Other:
- note added: "Battery Charging and power Distribution"
- note added: "ESP32 S3 Wroom 1 Microcontroler"
- note added: "Programmer"
- note added: "USB C"

Commit message: Going to bed.
Parts:
- removed D1 (x2): SS110, PCM_Diode_SMD_AKL:D_SMA, symbol PCM_Diode_Schottky_AKL:SS110
- removed P1: USB_C_Plug_USB2.0, symbol Connector:USB_C_Plug_USB2.0
- removed R1: 1.2k, PCM_Resistor_SMD_AKL:R_0603_1608Metric, symbol PCM_Resistor_AKL:R_0603
- removed R2, R3: 1k, PCM_Resistor_SMD_AKL:R_0603_1608Metric, symbol PCM_Resistor_AKL:R_0603
- removed TP1: Batt+, TestPoint:TestPoint_Pad_D1.0mm, symbol PCM_4ms_Connector:TestPoint
- removed TP2: Batt-, TestPoint:TestPoint_Pad_D1.0mm, symbol PCM_4ms_Connector:TestPoint
- removed U3: AMS1117-3.3, Package_TO_SOT_SMD:SOT-223-3_TabPin2, symbol Regulator_Linear:AMS1117-3.3
- added C1: 100nF, symbol Device:C_Small
- added C2: 10uF, symbol Device:C_Small
- added C? (x2): 1uF, symbol Device:C_Small
- added J?: USB_C_Receptacle_USB2.0_16P, symbol Connector:USB_C_Receptacle_USB2.0_16P
- added Q?: AO3401A, Package_TO_SOT_SMD:SOT-23, symbol Transistor_FET:AO3401A
- added R1, R2: 5.1kR, symbol Device:R_Small_US
- added R5: 10k, symbol Device:R_Small_US
- added R? (x2): 1kR, symbol Device:R_Small_US
- added R?: 1.2kR, symbol Device:R_Small_US
- added U4: ICM-45686, ICM-45686:IC_ICM-45686, symbol ICM-45686:ICM-45686
- added U?: AP2112K-3.3, Package_TO_SOT_SMD:SOT-23-5, symbol Regulator_Linear:AP2112K-3.3
- renumbered U4 to U3
Connections:
- net Data+: no longer U1.14 (USB_D+)
- net Data-: no longer U1.13 (USB_D-)
- net GND: now also C1.2, C2.2, C?.2, C?.2, J?.A1 (GND), J?.A12 (GND), J?.B1 (GND), J?.B12 (GND), J?.SH (SHIELD), R1.2, R2.2, R?.1, U4.6 (GND), U?.2 (GND)
- net VCC: no longer U2.4 (VCC)
- net at U2.2 (PROG): now also R?.2
- net at D3.1 (K): now also R?.2
- net at U2.6 (~{STDBY}): now also R?.1
- net at U2.7 (~{CHRG}): now also R?.1
- net VBUS: now reaches U2.8 (CE)
- net VBUS: now also U2.4 (VCC), C2.1, J?.A4 (VBUS), J?.A9 (VBUS), J?.B4 (VBUS), J?.B9 (VBUS)
- net at D2.1 (K): now also R?.2
- net IO17: now reaches U1.10 (IO17)
- net IO18: now reaches U1.11 (IO18)
- net IO8: now reaches U1.12 (IO8)
- net IO3: now reaches U1.15 (IO3)
- net IO46: now reaches U1.16 (IO46)
- net IO9: now reaches U1.17 (IO9)
- net IO10: now reaches U1.18 (IO10)
- net IO10: now also U4.12 (AP_CS)
- net IO11: now reaches U1.19 (IO11)
- net IO11: now also U4.14 (AP_SDA/AP_SDIO/AP_SDI)
- net IO12: now reaches U1.20 (IO12)
- net IO12: now also U4.13 (AP_SCL/AP_SCLK)
- net IO13: now reaches U1.21 (IO13)
- net IO14: now reaches U1.22 (IO14)
- net IO21: now reaches U1.23 (IO21)
- net IO47: now reaches U1.24 (IO47)
- net IO48: now reaches U1.25 (IO48)
- net IO45: now reaches U1.26 (IO45)
- net BOOT: now reaches U1.27 (IO0)
- net IO35: now reaches U1.28 (IO35)
- net IO36: now reaches U1.29 (IO36)
- net RESET: now reaches U1.3 (EN)
- net RESET: now also R5.2
- net IO37: now reaches U1.30 (IO37)
- net IO38: now reaches U1.31 (IO38)
- net IO39: now reaches U1.32 (IO39)
- net IO40: now reaches U1.33 (IO40)
- net IO41: now reaches U1.34 (IO41)
- net IO42: now reaches U1.35 (IO42)
- net RXD0: now reaches U1.36 (RXD0)
- net TXD0: now reaches U1.37 (TXD0)
- net IO2: now reaches U1.38 (IO2)
- net IO1: now reaches U1.39 (IO1)
- net IO4: now reaches U1.4 (IO4)
- net IO5: now reaches U1.5 (IO5)
- net IO6: now reaches U1.6 (IO6)
- net IO7: now reaches U1.7 (IO7)
- net IO15: now reaches U1.8 (IO15)
- net IO16: now reaches U1.9 (IO16)
- net Batt-v-read renamed VBAT
- net P,+3.3 renamed +3.3V
- net +3.3V: now also C1.1, C?.1, R5.1, U?.5 (VOUT)
- new net: J?.A5 (CC1), R2.1
- new net: J?.B5 (CC2), R1.1
- new net USB_D+: J?.A6 (D+), J?.B6 (D+), U1.14 (USB_D+)
- new net USB_D-: J?.A7 (D-), J?.B7 (D-), U1.13 (USB_D-)
- new net VIN: C?.1, U?.1 (VIN)
- no-connect marks 22 -> 20
Other:
- note added: "High-Current LDO"
- note added: "adfs"
- note removed: "Battery Charging and power Distribution"
- note removed: "Programmer"
- moved on the sheet: D2, D3, U1, U2, U3

Commit message: Taking a break
Parts:
- removed U3: CP2102N-Axx-xQFN28, Package_DFN_QFN:QFN-28-1EP_5x5mm_P0.5mm_EP3.35x3.35mm, symbol Interface_USB:CP2102N-Axx-xQFN28
- added C?: C_Small, symbol Device:C_Small
- added D?: 1N5819, Diode_THT:D_DO-41_SOD81_P10.16mm_Horizontal, symbol Diode:1N5819
- added J?: Conn_01x02, symbol Connector_Generic:Conn_01x02
- added R?: 100kR, symbol Device:R_Small_US
Connections:
- net GND: now also J?.1 (Pin_1), R?.1
- net VBAT: now also Q?.2 (S), J?.2 (Pin_2)
- net VBUS: now also Q?.1 (G), D?.1 (K), R?.2
- net VIN: now also Q?.3 (D), C?.2
- new net: C?.1, D?.2 (A)
- no-connect marks 20 -> 2
Other:
- note added: "Charging Manager"
- note added: "Load Sharing / Power Path"
- note removed: "adfs"
- moved on the sheet: C1, C?, D2, D3, Q?, R5, R?, U1, U2, U4, U?

Commit message: Did more work
Parts:
- added C? (x2): 0.1 uF, symbol Device:C_Small
Connections:
- net GND: now also C?.2, C?.2
- net IO10: no longer U4.12 (AP_CS)
- net IO11: no longer U4.14 (AP_SDA/AP_SDIO/AP_SDI)
- net IO12: no longer U4.13 (AP_SCL/AP_SCLK)
- net AP_AD0: now reaches U4.1 (AP_SDO/AP_AD0)
- net MAS_DA: now reaches U4.2 (RESV/AUX1_SDIO/AUX1_SDI/MAS_DA)
- net MAS_CLK: now reaches U4.3 (RESV/AUX1_SCLK/MAS_CLK)
- net INT1/INT: now reaches U4.4 (INT1/INT)
- net +3V3: now reaches U4.5 (VDDIO)
- net +3V3: now also U4.8 (VDD), C?.1, C?.1
- new net AP_CS: U4.12 (AP_CS)
- new net AP_SCL/AP_SCLK: U4.13 (AP_SCL/AP_SCLK)
- new net AP_SDA/AP_SDIO/AP_SDI: U4.14 (AP_SDA/AP_SDIO/AP_SDI)
- no-connect marks 2 -> 3
Other:
- note added: "I almost certainly know ts is very cooked"
- moved on the sheet: U4

Commit message: I should really figure out how pull-up resistors work
Parts:
- added R?: R_Small_US, symbol Device:R_Small_US
Connections:
- net IO10 is gone; now on net AP_CS: U1.18 (IO10)
- net IO11 is gone; now on net AP_SDA/AP_SDIO/AP_SDI: U1.19 (IO11)
- net IO12 is gone; now on net AP_SCL/AP_SCLK: U1.20 (IO12)
- net IO13 is gone; now on net RESV/AUX1_SDO: U1.21 (IO13)
- net IO14 is gone; now on net INT1/INT: U1.22 (IO14)
- net IO9 is gone; now on net INT2/FSYNC/CLKIN: U1.17 (IO9)
- net +3.3V: now also R?.2
- net INT1/INT: now also R?.1
- net RESV/AUX1_CS: now reaches U4.10 (RESV/AUX1_CS)
- net RESV/AUX1_SDO: now reaches U4.11 (RESV/AUX1_SDO)
- net INT2/FSYNC/CLKIN: now reaches U4.9 (INT2/FSYNC/CLKIN)
Other:
- moved on the sheet: C?

Commit message: label
Other:
- note added: "Gyro"
Changed lines of the file:
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@@
+		)
+	)
+	(rectangle
+		(start 67.31 95.25)
+		(end 184.15 207.01)
+		(stroke
+			(width 0)
+			(type default)
+		)
+		(fill
+			(type none)
 		)
 	)
@@
 		(effects
 			(font
+				(face "Times New Roman")
+				(size 3 3)
+				(color 255 0 0 1)
+			)
+		)
+	)
+	(text "Gyro"
+		(exclude_from_sim no)
+		(at 72.136 98.298 0)
+		(effects
+			(font

Commit message: new gyro
Parts:
- removed C? (x2): 0.1 uF, symbol Device:C_Small
- removed U4: ICM-45686, ICM-45686:IC_ICM-45686, symbol ICM-45686:ICM-45686
- added C3, C4: 0.1 uF, symbol Device:C_Small
- added R3, R4: 10k, symbol Device:R_Small_US
- added U3: LSM6DSV16XTR, LSM6DSV16XTR:XDCR_LSM6DSV16XTR, symbol LSM6DSV16XTR:LSM6DSV16XTR
Connections:
- net +3V3: now also C3.1, C4.1, R3.2, R4.2, U3.5 (VDD_IO), U3.8 (VDD)
- net GND: now also C3.2, C4.2, U3.6 (GND), U3.7 (GND)
- new net: R4.1, U3.1 (SDO/SA0)
- new net CS: R3.1, U3.12 (CS)
- new net INT1: U3.4 (INT1)
- new net INT2: U3.9 (INT2)
- new net OCS_AUX: U3.10 (OCS_AUX)
- new net SCL: U3.13 (SCL)
- new net SCX/AH2/QVAR2: U3.3 (SCX/AH2/QVAR2)
- new net SDA: U3.14 (SDA)
- new net SDO_AUX: U3.11 (SDO_AUX)
- new net SDX/AH1/QVAR1: U3.2 (SDX/AH1/QVAR1)
- no-connect marks 3 -> 2
Other:
- note added: "ESP32"
- note removed: "ESP32 S3 Wroom 1 Microcontroler"

Commit message: added gps
Parts:
- added C10, C11, C12, C5, C6, C7, C8, C9: C_Small, 21-0140_T2855+3_MXM, symbol Device:C_Small
- added R6: R_Small_US, Resistor_THT:R_Array_SIP4, symbol Device:R_Small_US
- added U4: MAX2769BETI/V+, 21-0140_T2855+3_MXM, symbol 2026-10-15_20-01-52:MAX2769BETI_V+
Connections:
- net GND: now also C10.2, C11.2, C12.2, C6.2, C7.2, C8.2, C9.2
- new net: C5.1, U4.2 (LNAOUT)
- new net: C5.2, U4.5 (MIXIN)
- new net: C9.1, R6.1
- new net: C10.1, R6.2, U4.12 (CPOUT)
- new net *IDLE: U4.24 (*IDLE)
- new net *SHDN: U4.7 (*SHDN)
- new net ANTBIAS: U4.3 (ANTBIAS)
- new net ANTFLAG: U4.1 (ANTFLAG)
- new net CLKOUT: U4.16 (CLKOUT)
- new net EP: U4.29 (EP)
- new net I0: U4.20 (I0)
- new net I1: U4.21 (I1)
- new net LD: U4.6 (LD)
- new net LNA1: U4.27 (LNA1)
- new net LNA2: U4.25 (LNA2)
- new net NC: U4.22 (NC), U4.28 (NC)
- new net PGM: U4.26 (PGM)
- new net Q0: U4.18 (Q0)
- new net Q1: U4.17 (Q1)
- new net VCCD: C11.1, U4.14 (VCCD)
- new net VCC_ADC: U4.19 (VCC_ADC)
- new net VCC_CP: C12.1, U4.13 (VCC_CP)
- new net VCC_IF: U4.23 (VCC_IF)
- new net VCC_RF: C6.1, C7.1, U4.4 (VCC_RF)
- new net VCC_VCO: C8.1, U4.11 (VCC_VCO)
- new net XTAL: U4.15 (XTAL)
- no-connect marks 2 -> 5
Other:
- note added: "GPS"
